File: electronics/midi-io/midi-io.kicad_pcb (KiCad board)
At the start: 2 copper layers, 20.5 x 26.5 mm, 11 parts, among them J1 MIDI, J2 HOST, U1 H11L1SR2M

Commit message: fixed pcb
Parts:
- J2: value HOST -> UART
Routing:
- net Net-(J1-Pin_1): track 10.9 -> 13.2 mm
Other:
- board text added: "+"
- board text added: "GND"
- board text added: "RX"
- board text added: "Rx"
- board text added: "TX"
- board text added: "Tx"
- board text added: "Vcc"
