File: electronics/midi-io/midi-io.kicad_sch (KiCad schematic)
At the start: 11 parts, among them J1 Conn_01x06, J2 Conn_01x06, U1 H11L1

Commit message: routed board
Parts:
- C1: LCSC (none) -> C14663
- D1: LCSC (none) -> C81598
- J1: value Conn_01x06 -> MIDI; footprint Connector_PinHeader_2.54mm:PinHeader_1x06_P2.54mm_Vertical -> Connector_Wire:SolderWire-0.25sqmm_1x06_P4.5mm_D0.65mm_OD2mm
- J2: value Conn_01x06 -> HOST; footprint Connector_JST:JST_XH_B6B-XH-A_1x06_P2.50mm_Vertical -> Connector_Wire:SolderWire-0.25sqmm_1x06_P4.5mm_D0.65mm_OD2mm
- R1: footprint Package_DIP:DIP-8_W7.62mm -> Resistor_SMD:R_0603_1608Metric; LCSC (none) -> C22962
- R2, R3: LCSC (none) -> C22962
- R4: LCSC (none) -> C23179
- U1: value H11L1 -> H11L1SR2M; LCSC (none) -> C20082
Changed lines of the file:
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@@
 			)
 		)
-		(property "Footprint" "RF_Mini-Circuits:Mini-Circuits_CK605_LandPatternPL-012"
+		(property "Footprint" ""
 			(at 120.65 69.85 0)
 			(hide yes)
@@
 			)
 		)
+		(property "LCSC" "C81598"
+			(at 165.1 78.74 0)
+			(hide yes)
+			(show_name no)
+			(do_not_autoplace no)
+			(effects
+				(font
+					(size 1.27 1.27)
+				)
+			)
+		)
 		(pin "2"
 		)
@@
 			)
 		)
-		(property "Footprint" "RF_Mini-Circuits:Mini-Circuits_CK605_LandPatternPL-012"
+		(property "Footprint" ""
 			(at 135.89 92.71 0)
 			(hide yes)
@@
 			)
 		)
+		(property "LCSC" "C23179"
+			(at 165.1 78.74 0)
+			(hide yes)
+			(show_name no)
+			(do_not_autoplace no)
+			(effects
+				(font
+					(size 1.27 1.27)
+				)
+			)
+		)
 		(pin "2"
 		)
@@
 			)
 		)
-		(property "Value" "H11L1"
+		(property "Value" "H11L1SR2M"
 			(at 130.81 73.5898 0)
 			(show_name no)
@@
 		(property "Description" "Schmitt Trigger Output Optocoupler, High Speed, DIP-6, 1.6mA turn on threshold"
 			(at 120.65 77.47 0)
+			(hide yes)
+			(show_name no)
+			(do_not_autoplace no)
+			(effects
+				(font
+					(size 1.27 1.27)
+				)
+			)
+		)
+		(property "LCSC" "C20082"
+			(at 118.364 77.47 0)
 			(hide yes)
 			(show_name no)
@@
 			)
 		)
+		(property "LCSC" "C22962"
+			(at 165.1 78.74 0)
+			(hide yes)
+			(show_name no)
+			(do_not_autoplace no)
+			(effects
+				(font
+					(size 1.27 1.27)
+				)
+			)
+		)
 		(pin "2"
 		)
@@
 		(property "Description" "Resistor"
 			(at 87.63 82.55 0)
+			(hide yes)
+			(show_name no)
+			(do_not_autoplace no)
+			(effects
+				(font
+					(size 1.27 1.27)
+				)
+			)
+		)
+		(property "LCSC" "C22962"
+			(at 87.63 84.328 0)
 			(hide yes)
 			(show_name no)
@@
 			)
 		)
+		(property "LCSC" "C14663"
+			(at 136.8552 100.33 0)
+			(hide yes)
+			(show_name no)
+			(do_not_autoplace no)
+			(effects
+				(font
+					(size 1.27 1.27)
+				)
+			)
+		)
 		(pin "2"
 		)
@@
 			)
 		)
-		(property "Footprint" "RF_Mini-Circuits:Mini-Circuits_CK605_LandPatternPL-012"
+		(property "Footprint" ""
 			(at 138.43 69.85 0)
 			(hide yes)
@@
 			)
 		)
-		(property "Value" "Conn_01x06"
+		(property "Value" "HOST"
 			(at 172.72 78.7399 0)
 			(show_name no)
@@
 			)
 		)
-		(property "Footprint" "Connector_JST:JST_XH_B6B-XH-A_1x06_P2.50mm_Vertical"
+		(property "Footprint" "Connector_Wire:SolderWire-0.25sqmm_1x06_P4.5mm_D0.65mm_OD2mm"
 			(at 170.18 76.2 0)
 			(hide yes)
@@
 			)
 		)
-		(property "Value" "Conn_01x06"
+		(property "Value" "MIDI"
 			(at 74.93 68.58 0)
 			(show_name no)
@@
 			)
 		)
-		(property "Footprint" "Connector_PinHeader_2.54mm:PinHeader_1x06_P2.54mm_Vertical"
+		(property "Footprint" "Connector_Wire:SolderWire-0.25sqmm_1x06_P4.5mm_D0.65mm_OD2mm"
 			(at 74.93 80.01 0)
 			(hide yes)
@@
 			)
 		)
-		(property "Footprint" "Package_DIP:DIP-8_W7.62mm"
+		(property "Footprint" "Resistor_SMD:R_0603_1608Metric"
 			(at 91.44 70.612 90)
 			(hide yes)
@@
 			(hide yes)
 			(show_name no)
+			(do_not_autoplace no)
+			(effects
+				(font
+					(size 1.27 1.27)
+				)
+			)
+		)
+		(property "LCSC" "C22962"
+			(at 165.1 78.74 0)
+			(hide yes)
+			(show_name no)

Commit message: fixed pcb
Parts:
- J2: value HOST -> MCU
Changed lines of the file:
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@@
 			)
 		)
-		(property "Value" "HOST"
+		(property "Value" "MCU"
 			(at 172.72 78.7399 0)
 			(show_name no)
